Commit message: catkin_make hecho

File: project_ws/src/VL/urdf/VL.xacro (robot description, xacro)
@@ -164,10 +164,10 @@
   </collision>
 </link>
-<joint name="R�gida1" type="fixed">
+<joint name="Rigida1" type="fixed">
   <origin xyz="0.0 0.0 0.07" rpy="0 0 0"/>
   <parent link="base_link"/>
   <child link="Componente5_1"/>
 </joint>
-<joint name="Revoluci�n2" type="revolute">
+<joint name="Revolucion2" type="revolute">
   <origin xyz="0.0 0.0 0.02" rpy="0 0 0"/>
   <parent link="Componente5_1"/>
@@ -176,5 +176,5 @@
   <limit upper="6.283185" lower="0.0" effort="100" velocity="100"/>
 </joint>
-<joint name="Revoluci�n3" type="revolute">
+<joint name="Revolucion3" type="revolute">
   <origin xyz="-0.0045 0.035737 0.036223" rpy="0 0 0"/>
   <parent link="q1_1"/>
@@ -183,5 +183,5 @@
   <limit upper="3.141593" lower="0.0" effort="100" velocity="100"/>
 </joint>
-<joint name="Revoluci�n4" type="revolute">
+<joint name="Revolucion4" type="revolute">
   <origin xyz="0.022 0.39 1.7e-05" rpy="0 0 0"/>
   <parent link="q2_1"/>
@@ -190,5 +190,5 @@
   <limit upper="6.283185" lower="0.0" effort="100" velocity="100"/>
 </joint>
-<joint name="Revoluci�n5" type="revolute">
+<joint name="Revolucion5" type="revolute">
   <origin xyz="-0.073 0.144 7e-06" rpy="0 0 0"/>
   <parent link="q3_1"/>
@@ -204,5 +204,5 @@
   <limit upper="0.24" lower="0.0" effort="100" velocity="100"/>
 </joint>
-<joint name="Revoluci�n7" type="revolute">
+<joint name="Revolucion7" type="revolute">
   <origin xyz="0.0 0.27 1.2e-05" rpy="0 0 0"/>
   <parent link="q5_1"/>

Commit message: v1

File: project_ws/src/VL/urdf/VL.xacro (robot description, xacro)
@@ -169,5 +169,5 @@
   <child link="Componente5_1"/>
 </joint>
-<joint name="Revolucion2" type="revolute">
+<joint name="shoulder_pan_joint" type="revolute">
   <origin xyz="0.0 0.0 0.02" rpy="0 0 0"/>
   <parent link="Componente5_1"/>
@@ -176,5 +176,5 @@
   <limit upper="6.283185" lower="0.0" effort="100" velocity="100"/>
 </joint>
-<joint name="Revolucion3" type="revolute">
+<joint name="shoulder_lift_joint" type="revolute">
   <origin xyz="-0.0045 0.035737 0.036223" rpy="0 0 0"/>
   <parent link="q1_1"/>
@@ -183,5 +183,5 @@
   <limit upper="3.141593" lower="0.0" effort="100" velocity="100"/>
 </joint>
-<joint name="Revolucion4" type="revolute">
+<joint name="elbow_joint" type="revolute">
   <origin xyz="0.022 0.39 1.7e-05" rpy="0 0 0"/>
   <parent link="q2_1"/>
@@ -190,5 +190,5 @@
   <limit upper="6.283185" lower="0.0" effort="100" velocity="100"/>
 </joint>
-<joint name="Revolucion5" type="revolute">
+<joint name="wrist_1_joint" type="revolute">
   <origin xyz="-0.073 0.144 7e-06" rpy="0 0 0"/>
   <parent link="q3_1"/>
@@ -197,5 +197,5 @@
   <limit upper="6.283185" lower="0.0" effort="100" velocity="100"/>
 </joint>
-<joint name="Corredera6" type="prismatic">
+<joint name="wrist_2_joint" type="prismatic">
   <origin xyz="-0.0265 0.085 3e-06" rpy="0 0 0"/>
   <parent link="q4_1"/>
@@ -204,5 +204,5 @@
   <limit upper="0.24" lower="0.0" effort="100" velocity="100"/>
 </joint>
-<joint name="Revolucion7" type="revolute">
+<joint name="wrist_3_joint" type="revolute">
   <origin xyz="0.0 0.27 1.2e-05" rpy="0 0 0"/>
   <parent link="q5_1"/>

Commit message: fkine e ikine

File: project_ws/src/VL/urdf/VL.xacro (robot description, xacro)
@@ -164,10 +164,10 @@
   </collision>
 </link>
-<joint name="Rigida1" type="fixed">
+<joint name="Rigida" type="fixed">
   <origin xyz="0.0 0.0 0.07" rpy="0 0 0"/>
   <parent link="base_link"/>
   <child link="Componente5_1"/>
 </joint>
-<joint name="shoulder_pan_joint" type="revolute">
+<joint name="waist_q1" type="revolute">
   <origin xyz="0.0 0.0 0.02" rpy="0 0 0"/>
   <parent link="Componente5_1"/>
@@ -176,5 +176,5 @@
   <limit upper="6.283185" lower="0.0" effort="100" velocity="100"/>
 </joint>
-<joint name="shoulder_lift_joint" type="revolute">
+<joint name="shoulder_q2" type="revolute">
   <origin xyz="-0.0045 0.035737 0.036223" rpy="0 0 0"/>
   <parent link="q1_1"/>
@@ -183,5 +183,5 @@
   <limit upper="3.141593" lower="0.0" effort="100" velocity="100"/>
 </joint>
-<joint name="elbow_joint" type="revolute">
+<joint name="revolution_q3" type="revolute">
   <origin xyz="0.022 0.39 1.7e-05" rpy="0 0 0"/>
   <parent link="q2_1"/>
@@ -190,5 +190,5 @@
   <limit upper="6.283185" lower="0.0" effort="100" velocity="100"/>
 </joint>
-<joint name="wrist_1_joint" type="revolute">
+<joint name="elbow_q4" type="revolute">
   <origin xyz="-0.073 0.144 7e-06" rpy="0 0 0"/>
   <parent link="q3_1"/>
@@ -197,5 +197,5 @@
   <limit upper="6.283185" lower="0.0" effort="100" velocity="100"/>
 </joint>
-<joint name="wrist_2_joint" type="prismatic">
+<joint name="slider_q5" type="prismatic">
   <origin xyz="-0.0265 0.085 3e-06" rpy="0 0 0"/>
   <parent link="q4_1"/>
@@ -204,5 +204,5 @@
   <limit upper="0.24" lower="0.0" effort="100" velocity="100"/>
 </joint>
-<joint name="wrist_3_joint" type="revolute">
+<joint name="wrist_q6" type="revolute">
   <origin xyz="0.0 0.27 1.2e-05" rpy="0 0 0"/>
   <parent link="q5_1"/>

Commit message: Se arregló problema en q5

File: project_ws/src/VL/urdf/VL.xacro (robot description, xacro)
@@ -174,5 +174,5 @@
   <child link="q1_1"/>
   <axis xyz="0.0 0.0 1.0"/>
-  <limit upper="6.283185" lower="0.0" effort="100" velocity="100"/>
+  <limit upper="3.141593" lower="-3.141593" effort="100" velocity="100"/>
 </joint>
 <joint name="shoulder_q2" type="revolute">
@@ -188,5 +188,5 @@
   <child link="q3_1"/>
   <axis xyz="-0.0 -1.0 -4.3e-05"/>
-  <limit upper="6.283185" lower="0.0" effort="100" velocity="100"/>
+  <limit upper="3.141593" lower="-3.141593" effort="100" velocity="100"/>
 </joint>
 <joint name="elbow_q4" type="revolute">
@@ -195,5 +195,5 @@
   <child link="q4_1"/>
   <axis xyz="-1.0 0.0 -0.0"/>
-  <limit upper="6.283185" lower="0.0" effort="100" velocity="100"/>
+  <limit upper="3.141593" lower="-3.141593" effort="100" velocity="100"/>
 </joint>
 <joint name="slider_q5" type="prismatic">
@@ -202,5 +202,5 @@
   <child link="q5_1"/>
   <axis xyz="0.0 1.0 4.3e-05"/>
-  <limit upper="0.24" lower="0.0" effort="100" velocity="100"/>
+  <limit upper="0.24" lower="0.00" effort="100" velocity="100"/>
 </joint>
 <joint name="wrist_q6" type="revolute">
@@ -209,5 +209,5 @@
   <child link="q6_1"/>
   <axis xyz="-0.0 -1.0 -4.3e-05"/>
-  <limit upper="6.283185" lower="0.0" effort="100" velocity="100"/>
+  <limit upper="3.141593" lower="-3.141593" effort="100" velocity="100"/>
 </joint>
 </robot>
